Commit message: Added better urdf file representation for robot, added ball indicator

File: scene/ufactory_xarm7/xarm7.urdf (robot description, URDF)
Before this commit: robot xarm7, 8 links, 7 joints
Links:
- link link7: geometry collision cylinder length=0.15 radius=0.003; collision mesh filename=assets/link7.stl

Commit message: Moved the ee from joint to end of the tool. Added method to change angles of tool

File: scene/ufactory_xarm7/xarm7.urdf (robot description, URDF)
Before this commit: robot None, 9 links, 8 joints
Joints:
- removed joint joint8
- added joint dummy_joint: type revolute, parent link7, child tool, origin xyz=0 0 0.3, axis 0 0 1, limit lower=0 upper=0 effort=1000 velocity=0.001
